File: pcb/PCB.sch (EAGLE design)
At the start: 17 parts

Commit message: Updated pcb
Parts:
- removed AND: 74HC21N, 74xx-eu:74HC21N
- added LED1, LED2, LED3: (no value), led:LEDSML0805
- added R5: 1k, resistor:R-US_R0805
- added R6, R7, R8: 100, resistor:R-US_R0805
- added U1: SN74LVC1G11DBVR, parts:SN74LVC1G11DBVR
- R1, R2: device resistor:R-US_0207/10 -> resistor:R-US_R0805
- R3, R4: value 200k -> 100k; device resistor:R-US_0207/10 -> resistor:R-US_R0805
- SV1: device parts:MA07-1 -> parts:MA08-1
Connections:
- new net N$2: LED3.C, R8.1
- new net N$3: R5.1, U1.Y
- new net N$5: LED2.C, R7.1
- new net N$6: LED1.C, R6.1
- new net NRST: MUX.PB5/PCINT5/!RESET!/ADC0/DW, SV1.8, UC1.PB5/PCINT5/!RESET!/ADC0/DW, UC2.PB5/PCINT5/!RESET!/ADC0/DW
- net 5V: now also OUT-GND.1, SV1.1; no longer SV1.7, T1.C
- net GND: now also R6.2, R7.2, R8.2, SV1.2, T1.E, U1.GND; no longer OUT-GND.2, SV1.1
- net HOT: now also LED3.A, SV1.7, U1.C; no longer ANDA.I2, SV1.6
- net MISO: now also SV1.4; no longer SV1.3
- net MOSI: now also SV1.5; no longer SV1.4
- net N$1: now also OUT-GND.2, T1.C; no longer OUT-GND.1, T1.E
- net N$4: now also R5.2; no longer ANDA.O
- net OUT1: now also LED1.A, U1.A; no longer ANDA.I1
- net OUT2: now also LED2.A, U1.B; no longer ANDA.I0
- net SCLK: now also SV1.3; no longer SV1.2
- net VCC: now also SV1.6, U1.VCC; no longer ANDA.I3, MUX.PB5/PCINT5/!RESET!/ADC0/DW, SV1.5, UC1.PB5/PCINT5/!RESET!/ADC0/DW, UC2.PB5/PCINT5/!RESET!/ADC0/DW
Other:
- moved on the sheet: H1, H3, MUX, OUT-GND, T1, UC1, UC2
